File: _autosave-ai03-PCB.kicad_pcb (KiCad board)
At the start: 2 copper layers, 24 parts, among them SW1 SW_Push, U1 ATmega32U4-A, Y1 16MHz

Commit message: Fix bugs in pcb design
Routing:
- net +5V: track 74.9 -> 76.2 mm
- net GND: track 17.9 -> 18.6 mm, vias 4 -> 5
Changed lines of the file:
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@@
         (effects (font (size 1 1) (thickness 0.15)))
     )
-    (fp_text value "22pF" (at -0.1016 1.7936 90) (layer "F.Fab")
+    (fp_text value "22pF" (at 0.1168 1.7936 90) (layer "F.Fab")
         (effects (font (size 1 1) (thickness 0.15)))
     )
@@
   (segment (start 211.2224 105.0696) (end 212.9224 106.7696) (width 0.25) (layer "F.Cu") (net 2))
   (via (at 215.138 92.1512) (size 0.8) (drill 0.4) (layers "F.Cu" "B.Cu") (free) (net 2))
-  (via (at 206.756 102.5144) (size 0.8) (drill 0.4) (layers "F.Cu" "B.Cu") (free) (net 2))
-  (via (at 224.4852 104.0892) (size 0.8) (drill 0.4) (layers "F.Cu" "B.Cu") (free) (net 2))
+  (via (at 206.6544 98.2472) (size 0.8) (drill 0.4) (layers "F.Cu" "B.Cu") (free) (net 2))
+  (via (at 221.6912 98.1964) (size 0.8) (drill 0.4) (layers "F.Cu" "B.Cu") (free) (net 2))
+  (via (at 209.8548 83.4136) (size 0.8) (drill 0.4) (layers "F.Cu" "B.Cu") (free) (net 2))
   (via (at 224.2312 85.09) (size 0.8) (drill 0.4) (layers "F.Cu" "B.Cu") (free) (net 2))
-  (segment (start 211.0232 89.154) (end 211.0232 90.4748) (width 0.25) (layer "B.Cu") (net 2))
   (segment (start 211.8868 96.0374) (end 211.8868 98.4504) (width 0.25) (layer "B.Cu") (net 2))
-  (segment (start 210.6168 88.7476) (end 211.0232 89.154) (width 0.25) (layer "B.Cu") (net 2))
-  (segment (start 210.6016 88.773) (end 210.6016 88.7628) (width 0.25) (layer "B.Cu") (net 2))
-  (segment (start 210.6016 88.7628) (end 210.6168 88.7476) (width 0.25) (layer "B.Cu") (net 2))
+  (segment (start 210.6016 88.773) (end 209.6008 89.7738) (width 0.25) (layer "B.Cu") (net 2))
+  (segment (start 209.6008 89.7738) (end 209.6008 90.9218) (width 0.25) (layer "B.Cu") (net 2))
   (segment (start 219.150105 86.7052) (end 221.3864 88.941495) (width 0.25) (layer "F.Cu") (net 3))
   (segment (start 207.7698 88.953) (end 207.5176 89.2052) (width 0.25) (layer "F.Cu") (net 3))
@@
   (segment (start 207.47162 87.531299) (end 207.7698 87.829479) (width 0.25) (layer "F.Cu") (net 3))
   (segment (start 219.6592 96.4692) (end 218.7952 95.6052) (width 0.25) (layer "F.Cu") (net 3))
+  (segment (start 208.297719 86.7052) (end 207.47162 87.531299) (width 0.25) (layer "F.Cu") (net 3))
   (segment (start 209.9564 99.3648) (end 209.9564 98.1436) (width 0.25) (layer "F.Cu") (net 3))
   (segment (start 218.7952 95.6052) (end 218.0948 95.6052) (width 0.25) (layer "F.Cu") (net 3))
   (segment (start 221.3864 88.941495) (end 221.3864 89.408) (width 0.25) (layer "F.Cu") (net 3))
+  (segment (start 208.3948 86.7052) (end 208.297719 86.7052) (width 0.25) (layer "F.Cu") (net 3))
   (segment (start 208.61688 94.3864) (end 209.6516 94.3864) (width 0.25) (layer "F.Cu") (net 3))
   (segment (start 216.3948 86.7052) (end 219.150105 86.7052) (width 0.25) (layer "F.Cu") (net 3))
