File: ai03-PCB.kicad_sch (KiCad schematic)
At the start: 24 parts, among them SW1 SW_Push, U1 ATmega32U4-A, Y1 16MHz

Commit message: Fix bugs in pcb design
Connections:
- net COL0: now also MX2.1 (COL), MX3.1 (COL), U1.29 (PB5); no longer MX1.1 (COL), MX4.1 (COL)
- net COL1: now also MX1.1 (COL), MX4.1 (COL), U1.28 (PB4); no longer MX2.1 (COL), MX3.1 (COL)
- net ROW0: now also D3.1 (K), D4.1 (K), U1.27 (PD7); no longer D1.1 (K), D2.1 (K)
- net ROW1: now also D1.1 (K), D2.1 (K), U1.30 (PB6); no longer D3.1 (K), D4.1 (K)
Changed lines of the file:
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@@
     (stroke (width 0) (type default))
   )
-  (global_label "COL0" (shape input) (at 179.07 66.04 90) (fields_autoplaced)
+  (global_label "COL0" (shape input) (at 194.31 66.04 90) (fields_autoplaced)
+    (effects (font (size 1.27 1.27)) (justify left))
+    (property "Intersheetrefs" "${INTERSHEET_REFS}" (at 194.31 58.2961 90)
+      (effects (font (size 1.27 1.27)) (justify left) hide)
+    )
+  )
+  (global_label "ROW0" (shape input) (at 163.83 100.33 180) (fields_autoplaced)
+    (effects (font (size 1.27 1.27)) (justify right))
+    (property "Intersheetrefs" "${INTERSHEET_REFS}" (at 155.6628 100.33 0)
+      (effects (font (size 1.27 1.27)) (justify right) hide)
+    )
+  )
+  (global_label "ROW0" (shape input) (at 124.46 101.6 0) (fields_autoplaced)
+    (effects (font (size 1.27 1.27)) (justify left))
+    (property "Intersheetrefs" "${INTERSHEET_REFS}" (at 132.6272 101.6 0)
+      (effects (font (size 1.27 1.27)) (justify left) hide)
+    )
+  )
+  (global_label "COL1" (shape input) (at 179.07 66.04 90) (fields_autoplaced)
     (effects (font (size 1.27 1.27)) (justify left))
     (property "Intersheetrefs" "${INTERSHEET_REFS}" (at 179.07 58.2961 90)
@@
     )
   )
-  (global_label "ROW0" (shape input) (at 163.83 85.09 180) (fields_autoplaced)
+  (global_label "ROW1" (shape input) (at 124.46 68.58 0) (fields_autoplaced)
+    (effects (font (size 1.27 1.27)) (justify left))
+    (property "Intersheetrefs" "${INTERSHEET_REFS}" (at 132.6272 68.58 0)
+      (effects (font (size 1.27 1.27)) (justify left) hide)
+    )
+  )
+  (global_label "COL1" (shape input) (at 124.46 63.5 0) (fields_autoplaced)
+    (effects (font (size 1.27 1.27)) (justify left))
+    (property "Intersheetrefs" "${INTERSHEET_REFS}" (at 132.2039 63.5 0)
+      (effects (font (size 1.27 1.27)) (justify left) hide)
+    )
+  )
+  (global_label "D-" (shape input) (at 46.99 147.32 0) (fields_autoplaced)
+    (effects (font (size 1.27 1.27)) (justify left))
+    (property "Intersheetrefs" "${INTERSHEET_REFS}" (at 52.7382 147.32 0)
+      (effects (font (size 1.27 1.27)) (justify left) hide)
+    )
+  )
+  (global_label "COL0" (shape input) (at 124.46 66.04 0) (fields_autoplaced)
+    (effects (font (size 1.27 1.27)) (justify left))
+    (property "Intersheetrefs" "${INTERSHEET_REFS}" (at 132.2039 66.04 0)
+      (effects (font (size 1.27 1.27)) (justify left) hide)
+    )
+  )
+  (global_label "ROW1" (shape input) (at 163.83 85.09 180) (fields_autoplaced)
     (effects (font (size 1.27 1.27)) (justify right))
     (property "Intersheetrefs" "${INTERSHEET_REFS}" (at 155.6628 85.09 0)
-      (effects (font (size 1.27 1.27)) (justify right) hide)
-    )
-  )
-  (global_label "COL1" (shape input) (at 194.31 66.04 90) (fields_autoplaced)
-    (effects (font (size 1.27 1.27)) (justify left))
-    (property "Intersheetrefs" "${INTERSHEET_REFS}" (at 194.31 58.2961 90)
-      (effects (font (size 1.27 1.27)) (justify left) hide)
-    )
-  )
-  (global_label "D-" (shape input) (at 46.99 147.32 0) (fields_autoplaced)
-    (effects (font (size 1.27 1.27)) (justify left))
-    (property "Intersheetrefs" "${INTERSHEET_REFS}" (at 52.7382 147.32 0)
-      (effects (font (size 1.27 1.27)) (justify left) hide)
-    )
-  )
-  (global_label "ROW1" (shape input) (at 163.83 100.33 180) (fields_autoplaced)
-    (effects (font (size 1.27 1.27)) (justify right))
-    (property "Intersheetrefs" "${INTERSHEET_REFS}" (at 155.6628 100.33 0)
       (effects (font (size 1.27 1.27)) (justify right) hide)
     )
@@
   )
   (symbol (lib_id "Device:R_Small_US") (at 131.445 106.68 270) (unit 1)
-    (in_bom yes) (on_board yes) (dnp no) (fields_autoplaced)
-    (property "Reference" "R1" (at 131.445 101.6 90)
-      (effects (font (size 1.27 1.27)))
-    )
-    (property "Value" "10k" (at 131.445 104.14 90)
-      (effects (font (size 1.27 1.27)))
-    )
+    (in_bom yes) (on_board yes) (dnp no)
+    (property "Reference" "R1" (at 128.27 104.14 90)
+      (effects (font (size 1.27 1.27)))
+    )
+    (property "Value" "10k" (at 133.35 104.14 90)
+      (effects (font (size 1.27 1.27)))
+    )
